File: shield/env_mapper_shield.kicad_pcb (KiCad board)
At the start: 2 copper layers, 70 x 57.5 mm, 5 parts, among them J1 CN7, J2 CN10

Commit message: shield redo + gitignore update
Parts:
- removed H1, H2, H3: MountingHole, MountingHole:MountingHole_3.2mm_M3
- added J3: Analog, Connector_PinSocket_2.54mm:PinSocket_1x06_P2.54mm_Vertical, F.Cu at (150.8, 97.5)
- added J4: Digital/PWM, Connector_PinSocket_2.54mm:PinSocket_1x08_P2.54mm_Vertical, F.Cu at (145.7, 49.2)
- added MH1: MountingHole_3.2mm, Arduino_MountingHole:MountingHole_3.2mm, F.Cu at (115.2, 49.2)
- added MH2: MountingHole_3.2mm, Arduino_MountingHole:MountingHole_3.2mm, F.Cu at (114.0, 97.5)
- added MH3: MountingHole_3.2mm, Arduino_MountingHole:MountingHole_3.2mm, F.Cu at (166.0, 64.4)
- added MH4: MountingHole_3.2mm, Arduino_MountingHole:MountingHole_3.2mm, F.Cu at (166.0, 92.4)
- J1: value CN7 -> Power; footprint Connector_PinSocket_2.54mm:PinSocket_2x19_P2.54mm_Vertical -> Connector_PinSocket_2.54mm:PinSocket_1x08_P2.54mm_Vertical; moved to F.Cu
- J2: value CN10 -> Digital/PWM; footprint Connector_PinSocket_2.54mm:PinSocket_2x19_P2.54mm_Vertical -> Connector_PinSocket_2.54mm:PinSocket_1x10_P2.54mm_Vertical; moved to F.Cu
- moved J2 48.7 mm to (118.8, 49.2), turned to 90 degrees
- moved J1 42.2 mm to (127.9, 97.5), turned to 90 degrees
Connections:
- net /5V_USB_CHGR renamed /*10
- J1 pad 2: unconnected-(J1-Pin_2-Pad2) -> /IOREF
- J1 pad 3: unconnected-(J1-Pin_3-Pad3) -> /~{RESET}
- J1 pad 4: unconnected-(J1-Pin_4-Pad4) -> +3V3
- J1 pad 5: VDD -> +5V
- J1 pad 6: /E5V -> GND
- J1 pad 7: unconnected-(J1-Pin_7-Pad7) -> GND
- J1 pad 8: GND -> VCC
- J2 pad 1: unconnected-(J2-Pin_1-Pad1) -> /SCL/A5
- J2 pad 10: unconnected-(J2-Pin_10-Pad10) -> /8
- J2 pad 2: unconnected-(J2-Pin_2-Pad2) -> /SDA/A4
- J2 pad 3: unconnected-(J2-Pin_3-Pad3) -> /AREF
- J2 pad 4: unconnected-(J2-Pin_4-Pad4) -> GND
- J2 pad 5: unconnected-(J2-Pin_5-Pad5) -> /13
- J2 pad 6: unconnected-(J2-Pin_6-Pad6) -> /12
- J2 pad 7: unconnected-(J2-Pin_7-Pad7) -> /*11
- J2 pad 9: unconnected-(J2-Pin_9-Pad9) -> /*9
Other:
- board size 70 x 57.5 mm -> 68.6 x 53.3 mm
- board text added: "ICSP"

Commit message: PCB layout started
Parts:
- added C1: 2.2uF, Resistor_SMD:R_0402_1005Metric_Pad0.72x0.64mm_HandSolder, F.Cu at (109.0, 79.0)
- added C2: 0.1uF, Resistor_SMD:R_0402_1005Metric_Pad0.72x0.64mm_HandSolder, F.Cu at (106.8, 76.0)
- added C3: 100uF, Capacitor_THT:CP_Radial_D8.0mm_P3.50mm, F.Cu at (146.8, 58.0)
- added C4: 0.1uF, Resistor_SMD:R_0402_1005Metric_Pad0.72x0.64mm_HandSolder, F.Cu at (164.0, 55.5)
- added C5: 0.1uF, Resistor_SMD:R_0402_1005Metric_Pad0.72x0.64mm_HandSolder, F.Cu at (155.0, 55.5)
- added C6: 0.1uF, Resistor_SMD:R_0402_1005Metric_Pad0.72x0.64mm_HandSolder, F.Cu at (163.0, 86.0)
- added C7: 22uF, Capacitor_SMD:C_0805_2012Metric_Pad1.18x1.45mm_HandSolder, F.Cu at (113.2, 76.2)
- added C8: 22uF, Capacitor_SMD:C_0805_2012Metric_Pad1.18x1.45mm_HandSolder, F.Cu at (115.5, 76.2)
- added IC2: PJ-002A, SamacSys_Parts:PJ002A, F.Cu at (113.0, 86.0)
- added J5: Pan, Connector_PinHeader_2.54mm:PinHeader_1x03_P2.54mm_Vertical, F.Cu at (161.5, 55.0)
- added J6: Tilt, Connector_PinHeader_2.54mm:PinHeader_1x03_P2.54mm_Vertical, F.Cu at (157.5, 55.0)
- added J7: LiDAR, Connector_PinSocket_2.54mm:PinSocket_1x04_P2.54mm_Vertical, F.Cu at (165.5, 79.5)
- added J8: E5V, Connector_PinHeader_2.54mm:PinHeader_1x01_P2.54mm_Vertical, F.Cu at (122.2, 97.5)
- added L1: 6.8uH, SamacSys_Parts:ETQ-P3M_KVP, F.Cu at (110.0, 70.2)
- added PS1: LMR51430XDDCR, SamacSys_Parts:SOT95P280X110-6N, F.Cu at (109.0, 76.2)
- added R1: 13.7k, Resistor_SMD:R_0402_1005Metric_Pad0.72x0.64mm_HandSolder, F.Cu at (111.5, 77.6)
- added R2: 100k, Resistor_SMD:R_0402_1005Metric_Pad0.72x0.64mm_HandSolder, F.Cu at (111.5, 75.2)
Connections:
- J1 pad 8: VCC -> GND
- J4 pad 2: /*6 -> Net-(J4-Pin_2)
- J4 pad 3: /*5 -> Net-(J4-Pin_3)
Routing:
- net Net-(J5-Pin_2): track 0.00 -> 148.3 mm
- net /RX/0: track 0.00 -> 36.3 mm
- net /TX/1: track 0.00 -> 33.5 mm
- net Net-(J4-Pin_3): track 0.00 -> 25.4 mm
- net GND: track 0.00 -> 24.3 mm, vias 0 -> 7
- net Net-(J4-Pin_2): track 0.00 -> 18.9 mm
- net Net-(PS1-EN): track 0.00 -> 12.9 mm, vias 0 -> 1
- net Net-(PS1-SW): track 0.00 -> 11.5 mm
- net Net-(PS1-FB): track 0.00 -> 1.73 mm
- net Net-(PS1-CB): track 0.00 -> 1.47 mm
- added copper zone on B.Cu, net GND
Other:
- board text added: "E5V"
- board text added: "LiDAR"
- board text added: "Pan"
- board text added: "Tilt"
