File: shield/env_mapper_shield.kicad_sch (KiCad schematic)
At the start: 5 parts, among them J1 CN7, J2 CN10

Commit message: shield redo + gitignore update
Parts:
- removed H1, H2, H3: MountingHole, MountingHole:MountingHole_3.2mm_M3, symbol Mechanical:MountingHole
- removed J1: CN7, Connector_PinSocket_2.54mm:PinSocket_2x19_P2.54mm_Vertical, symbol Connector_Generic:Conn_02x19_Odd_Even
- removed J2: CN10, Connector_PinSocket_2.54mm:PinSocket_2x19_P2.54mm_Vertical, symbol Connector_Generic:Conn_02x19_Odd_Even
- added IC1: MC78LC50NTRG, SamacSys_Parts:MC78LC50NTRG, symbol Library Loader:MC78LC50NTRG
- added IC2: PJ-002A, SamacSys_Parts:PJ002A, symbol Library Loader:PJ-002A
- added J1: Power, Connector_PinSocket_2.54mm:PinSocket_1x08_P2.54mm_Vertical, symbol Connector_Generic:Conn_01x08
- added J2: Digital/PWM, Connector_PinSocket_2.54mm:PinSocket_1x10_P2.54mm_Vertical, symbol Connector_Generic:Conn_01x10
- added J3: Analog, Connector_PinSocket_2.54mm:PinSocket_1x06_P2.54mm_Vertical, symbol Connector_Generic:Conn_01x06
- added J4: Digital/PWM, Connector_PinSocket_2.54mm:PinSocket_1x08_P2.54mm_Vertical, symbol Connector_Generic:Conn_01x08
Connections:
- net +3V3: now also J1.4 (Pin_4)
- net +5V: now also J1.5 (Pin_5)
- net GND: now also IC1.1 (GND), IC2.2, J1.6 (Pin_6), J1.7 (Pin_7), J2.4 (Pin_4)
- net IOREF: now also J1.2 (Pin_2)
- new net: IC1.2 (VIN), IC2.1
- new net *10: J2.8 (Pin_8)
- new net *11: J2.7 (Pin_7)
- new net *3: J4.5 (Pin_5)
- new net *5: J4.3 (Pin_3)
- new net *6: J4.2 (Pin_2)
- new net *9: J2.9 (Pin_9)
- new net 12: J2.6 (Pin_6)
- new net 13: J2.5 (Pin_5)
- new net 2: J4.6 (Pin_6)
- new net 4: J4.4 (Pin_4)
- new net 7: J4.1 (Pin_1)
- new net 8: J2.10 (Pin_10)
- new net A0: J3.1 (Pin_1)
- new net A1: J3.2 (Pin_2)
- new net A2: J3.3 (Pin_3)
- new net A3: J3.4 (Pin_4)
- new net AREF: J2.3 (Pin_3)
- new net RX/0: J4.8 (Pin_8)
- new net SCL/A5: J2.1 (Pin_1), J3.6 (Pin_6)
- new net SDA/A4: J2.2 (Pin_2), J3.5 (Pin_5)
- new net TX/1: J4.7 (Pin_7)
- new net VCC: J1.8 (Pin_8)
- new net ~{RESET}: J1.3 (Pin_3)
- no-connect marks 0 -> 1
Other:
- note added: "* Indicates a PWM-capable pin"
- note removed: "Mechanical"

Commit message: Shield completed, pending verification
Parts:
- removed IC1: MC78LC50NTRG, SamacSys_Parts:MC78LC50NTRG, symbol Library Loader:MC78LC50NTRG
- added C2: 100uF, Capacitor_THT:CP_Radial_D6.3mm_P2.50mm, symbol Device:C_Polarized
- added C3: 1000uF, Capacitor_THT:CP_Radial_D6.3mm_P2.50mm, symbol Device:C_Polarized
- added C4, C5, C6: 0.1uF, Capacitor_SMD:C_1206_3216Metric_Pad1.33x1.80mm_HandSolder, symbol Device:C
- added D1: LED, LED_SMD:LED_0201_0603Metric_Pad0.64x0.40mm_HandSolder, symbol Device:LED
- added D3: 1N5822, Diode_THT:D_DO-201AD_P15.24mm_Horizontal, symbol Diode:1N5822
- added IC1: LM2576S-5.0_NOPB, SamacSys_Parts:KTT0005B, symbol Library Loader:LM2576S-5.0_NOPB
- added J5: Pan_Servo, Connector_PinHeader_2.54mm:PinHeader_1x03_P2.54mm_Vertical, symbol Connector:Conn_01x03_Pin
- added J6: Tilt_Servo, Connector_PinHeader_2.54mm:PinHeader_1x03_P2.54mm_Vertical, symbol Connector:Conn_01x03_Pin
- added J7: LiDAR, Connector_PinSocket_2.54mm:PinSocket_1x04_P2.54mm_Vertical, symbol Connector:Conn_01x04_Socket
- added J8: E5V, Connector_PinHeader_2.54mm:PinHeader_1x01_P2.54mm_Vertical, symbol Connector:Conn_01x01_Socket
- added L1: 100uH, symbol Device:L
- added R1: 330ohm, Resistor_SMD:R_1206_3216Metric_Pad1.30x1.75mm_HandSolder, symbol Device:R
Connections:
- net VCC is gone; now on net GND: J1.8 (Pin_8)
- net GND: now also IC2.3, C2.2, C3.2, C4.2, C5.2, C6.2, D3.2 (A), IC1.3 (GND_1), IC1.5 (~{ON}/OFF), IC1.6 (GND_2), J5.3 (Pin_3), J6.3 (Pin_3), J7.4 (Pin_4)
- net RX/0: now also J7.2 (Pin_2)
- net TX/1: now also J7.1 (Pin_1)
- net at IC2.1: now also C2.1, IC1.1 (VIN)
- net *5: no longer names the net of J4.3 (Pin_3)
- net *5: now also C5.1, J6.1 (Pin_1)
- net *6: no longer names the net of J4.2 (Pin_2)
- net *6: now also C6.1, J5.1 (Pin_1)
- new net: D3.1 (K), IC1.2 (OUTPUT), L1.2
- new net: C3.1, IC1.4 (FEEDBACK), L1.1, R1.2
- new net: C4.1, D1.1 (K), J5.2 (Pin_2), J6.2 (Pin_2), J7.3 (Pin_3), J8.1 (Pin_1)
- new net: D1.2 (A), R1.1
Other:
- moved on the sheet: IC2

Commit message: Shield updates
Other:
- title: (none) -> Environment Mapper Shield
Changed lines of the file:
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@@
 	(paper "A4")
 	(title_block
+		(title "Environment Mapper Shield")
 		(date "mar. 31 mars 2015")
+		(rev "v1.0.0")
 	)
 	(text "* Indicates a PWM-capable pin"

Commit message: PCB layout started
Parts:
- removed C2: 100uF, Capacitor_THT:CP_Radial_D6.3mm_P2.50mm, symbol Device:C_Polarized
- removed D1: LED, LED_SMD:LED_0201_0603Metric_Pad0.64x0.40mm_HandSolder, symbol Device:LED
- removed D3: 1N5822, Diode_THT:D_DO-201AD_P15.24mm_Horizontal, symbol Diode:1N5822
- removed IC1: LM2576S-5.0_NOPB, SamacSys_Parts:KTT0005B, symbol Library Loader:LM2576S-5.0_NOPB
- added C1: 2.2uF, Resistor_SMD:R_0402_1005Metric_Pad0.72x0.64mm_HandSolder, symbol Device:C
- added C2: 0.1uF, Resistor_SMD:R_0402_1005Metric_Pad0.72x0.64mm_HandSolder, symbol Device:C
- added C7, C8: 22uF, Capacitor_SMD:C_0805_2012Metric_Pad1.18x1.45mm_HandSolder, symbol Device:C
- added PS1: LMR51430XDDCR, SamacSys_Parts:SOT95P280X110-6N, symbol Library Loader:LMR51430XDDCR
- added R2: 100k, Resistor_SMD:R_0402_1005Metric_Pad0.72x0.64mm_HandSolder, symbol Device:R
- C3: value 1000uF -> 100uF; footprint Capacitor_THT:CP_Radial_D6.3mm_P2.50mm -> Capacitor_THT:CP_Radial_D8.0mm_P3.50mm
- C4, C5, C6: footprint Capacitor_SMD:C_1206_3216Metric_Pad1.33x1.80mm_HandSolder -> Resistor_SMD:R_0402_1005Metric_Pad0.72x0.64mm_HandSolder
- L1: value 100uH -> 6.8uH; footprint (none) -> SamacSys_Parts:ETQ-P3M_KVP
- R1: value 330ohm -> 13.7k; footprint Resistor_SMD:R_1206_3216Metric_Pad1.30x1.75mm_HandSolder -> Resistor_SMD:R_0402_1005Metric_Pad0.72x0.64mm_HandSolder
Connections:
- net GND: now also R1.1, C1.2, C7.1, C8.1, PS1.1 (GND)
- net at J4.2 (Pin_2), J5.1 (Pin_1): now also C4.1; no longer C6.1
- net at L1.2: now also C2.1, PS1.2 (SW)
- net at IC2.1: now also C1.1, PS1.3 (VIN), PS1.5 (EN)
- net at C3.1, L1.1, R1.2: now also C6.1, J5.2 (Pin_2), J6.2 (Pin_2), J7.3 (Pin_3), J8.1 (Pin_1), C7.2, C8.2, R2.1
- new net: PS1.4 (FB), R2.2
- new net: C2.2, PS1.6 (CB)
Other:
- moved on the sheet: IC2
